File: KICAD/PW_Cond.kicad_pcb (KiCad board)
At the start: 2 copper layers, 30 x 30 mm, 26 parts, among them J1 Conn_01x02_Female, J2 Conn_01x04_Female, J3 Conn_01x02_Female, Q1 BC847, U1 MCP602, U2 MCP602

Commit message: cleanup + fab files wip
Routing:
- net Net-(D1-Pad1): track 27.4 -> 14.5 mm
- net +15V: track 58.3 -> 60.3 mm, vias 2 -> 3
- net GND: vias 28 -> 27
